Commit message: Upload URDF file: sa2000h_urdf_0521.urdf

File: jobs/current/robot.urdf (robot description, URDF)
Before this commit: robot 6dof_arm, 8 links, 7 joints
Links:
- removed link ee_link
- removed link forearm_link
- removed link shoulder_link
- removed link upper_arm_link
- removed link wrist_1_link
- removed link wrist_2_link
- removed link wrist_3_link
- added link link1, mass 0.1259; collision mesh filename=package://sa2000h_urdf_0521/meshes/link1.STL; visual mesh filename=package://sa2000h_urdf_0521/meshes/link1.STL
- added link link2, mass 0.062211; collision mesh filename=package://sa2000h_urdf_0521/meshes/link2.STL; visual mesh filename=package://sa2000h_urdf_0521/meshes/link2.STL
- added link link3, mass 0.11857; collision mesh filename=package://sa2000h_urdf_0521/meshes/link3.STL; visual mesh filename=package://sa2000h_urdf_0521/meshes/link3.STL
- added link link4, mass 0.087667; collision mesh filename=package://sa2000h_urdf_0521/meshes/link4.STL; visual mesh filename=package://sa2000h_urdf_0521/meshes/link4.STL
- added link link5, mass 0.0080739; collision mesh filename=package://sa2000h_urdf_0521/meshes/link5.STL; visual mesh filename=package://sa2000h_urdf_0521/meshes/link5.STL
- added link link6, mass 1.4715; collision mesh filename=package://sa2000h_urdf_0521/meshes/link6.STL; visual mesh filename=package://sa2000h_urdf_0521/meshes/link6.STL
- added link link_flp; collision box size=0.0001 0.0001 0.0001
- added link link_tool
- link base_link: mass 2.0 -> None; geometry collision mesh filename=package://sa2000h_urdf_0521/meshes/base_link.STL; visual mesh filename=package://sa2000h_urdf_0521/meshes/base_link.STL
Joints:
- removed joint ee_joint
- removed joint elbow_joint
- removed joint shoulder_lift_joint
- removed joint shoulder_pan_joint
- removed joint wrist_1_joint
- removed joint wrist_2_joint
- removed joint wrist_3_joint
- added joint joint1: type revolute, parent base_link, child link1, origin xyz=0 0 0.421 rpy=0 0 0, axis 0 0 -1, limit lower=-2.8798 upper=2.8798 effort=0 velocity=0
- added joint joint2: type revolute, parent link1, child link2, origin xyz=0.19 0 0 rpy=1.5708 -1.5708 0, axis 0 0 -1, limit lower=-1.3963 upper=2.8449 effort=0 velocity=0
- added joint joint3: type revolute, parent link2, child link3, origin xyz=0.765 0 0 rpy=0 0 0, axis 0 0 -1, limit lower=-1.3963 upper=1.3963 effort=0 velocity=0
- added joint joint4: type revolute, parent link3, child link4, origin xyz=0.2 -1.0365 0 rpy=1.5708 0 0, axis 0 0 -1, limit lower=-1.6 upper=1.6 effort=0 velocity=0
- added joint joint5: type revolute, parent link4, child link5, origin xyz=0 0 0 rpy=1.5708 1.5708 0, axis 0 0 1, limit lower=-2.2689 upper=2.2689 effort=0 velocity=0
- added joint joint6: type revolute, parent link5, child link6, origin xyz=0 0 0 rpy=1.5708 0 -1.5708, axis 0 0 -1, limit lower=-6.2832 upper=6.2832 effort=0 velocity=0
- added joint joint_flp: type fixed, parent link6, child link_flp, origin xyz=0 0 0.1 rpy=0 0 3.1415926
- added joint joint_tool: type fixed, parent link_flp, child link_tool, origin xyz=-0.078526107 -0.001290739 0.429874408 rpy=0.028969707963 0.554835928059 -3.111924552127
